Commit message: feat(logistics): replace cargo proxies with AWS source CAD and detail warehouse bays

File: assets/world/native-logistics.urdf (robot description, URDF)
Before this commit: robot delivery_logistics_visual, 1 links, 0 joints
Links:
- link odom: geometry visual box size=0.075 1.17 0.012; visual box size=0.075 1.17 0.012
